File: Wideband-Test-V1.kicad_pcb (KiCad board)
At the start: 4 copper layers, 120 x 110 mm, 215 parts, among them IC1 LMX2592RHAT, IC2 BU7205HFV-TR, IC3 GRF3042, IC4 OPA2673IRGVR, IC5 BU7205HFV-TR, IC6 BU7205HFV-TR, IC7 OPA2673IRGVR, IC8 OPA2673IRGVR, IC9 OPA2673IRGVR, J1 Conn_01x02_Pin, J2 Conn_01x02_Pin, J3 Conn_01x04_Pin, P1 USB_C_Plug, Q1 MMBFJ113, Q10 MMBFJ113, Q11 MMBFJ113, Q12 BFP840ESD, Q13 BFP840ESD, Q14 BFP840ESD, Q15 BFP840ESD, Q16 BFP840ESD, Q2 MMBFJ113, Q3 MMBFJ113, Q4 MMBFJ113, Q5 MMBFJ113, Q6 MMBFJ113, Q7 BFP840ESD, Q8 MMBFJ113, Q9 MMBFJ113, T1 CX2041NLT, U1 AD9215BCPZ-105, U2 BGA614H6327XTSA1, U3 LD1117V-3V3, U4 BGA614H6327XTSA1, U5 AP7381-50SA-7, U6 DSP, Y1 Crystal_GND24

Commit message: 1.x
Parts:
- removed ? (x2): , 
- removed D1, D10, D11, D12, D13, D2, D3, D4, D5, D6, D7, D8, D9: MMBZ15VAL215, Package_TO_SOT_SMD:SOT-323_SC-70
- removed IC8, IC9: OPA2673IRGVR, Package_DFN_QFN:QFN-16-1EP_4x4mm_P0.65mm_EP2.1x2.1mm_ThermalVias
- removed L2: 10u, Inductor_SMD:L_0603_1608Metric
- removed P1: USB_C_Plug, Connector_USB:USB_C_Receptacle_Molex_105450-0101
- removed T1: CX2041NLT, KiCad:CX2041NLT
- added C103: 0.1uF, Capacitor_SMD:C_0603_1608Metric, F.Cu at (130.3, 18.9)
- added C104: 10uF, Capacitor_SMD:C_0603_1608Metric, F.Cu at (130.3, 21.5)
- added C105: 22uF, Capacitor_SMD:C_1206_3216Metric, F.Cu at (144.0, 55.4)
- added C106: 1nF, Capacitor_SMD:C_0402_1005Metric, F.Cu at (158.4, 11.2)
- added C107: 22uF, Capacitor_SMD:C_1206_3216Metric, F.Cu at (144.0, 58.7)
- added C108: 0.1uF, Capacitor_SMD:C_0603_1608Metric, F.Cu at (130.3, 24.0)
- added C109: 1nF, Capacitor_SMD:C_0402_1005Metric, F.Cu at (158.4, 13.1)
- added C110: 10uF, Capacitor_SMD:C_0603_1608Metric, F.Cu at (130.3, 26.5)
- added C111: 0.1uF, Capacitor_SMD:C_0603_1608Metric, F.Cu at (130.3, 29.0)
- added C112: 0.1uF, Capacitor_SMD:C_0603_1608Metric, F.Cu at (130.3, 31.5)
- added C113: 10uF, Capacitor_SMD:C_0603_1608Metric, F.Cu at (130.3, 34.0)
- added C114: 0.1uF, Capacitor_SMD:C_0603_1608Metric, F.Cu at (130.3, 36.5)
- added C115: 0.1uF, Capacitor_SMD:C_0603_1608Metric, F.Cu at (130.3, 39.0)
- added C116: 0.1uF, Capacitor_SMD:C_0603_1608Metric, F.Cu at (130.3, 41.5)
- added C117: 0.1uF, Capacitor_SMD:C_0603_1608Metric, F.Cu at (130.3, 44.0)
- added C118: 1nF, Capacitor_SMD:C_0402_1005Metric, F.Cu at (158.4, 15.1)
- added C119: 1nF, Capacitor_SMD:C_0402_1005Metric, F.Cu at (158.4, 17.1)
- added C120: 100pF, Capacitor_SMD:C_0603_1608Metric, F.Cu at (130.3, 46.6)
- added C121: 30pF, Capacitor_SMD:C_0603_1608Metric, F.Cu at (130.3, 49.1)
- added C122: 30pF, Capacitor_SMD:C_0603_1608Metric, F.Cu at (134.3, 11.4)
- added C123: 30pF, Capacitor_SMD:C_0603_1608Metric, F.Cu at (134.3, 13.9)
- added C124: 30pF, Capacitor_SMD:C_0603_1608Metric, F.Cu at (134.3, 16.4)
- added C125: 10uF, Capacitor_SMD:C_0603_1608Metric, F.Cu at (134.3, 18.9)
- added C126: 10uF, Capacitor_SMD:C_0603_1608Metric, F.Cu at (134.3, 21.5)
- added C127: 1nF, Capacitor_SMD:C_0402_1005Metric, F.Cu at (158.4, 19.0)
- added C128: 1nF, Capacitor_SMD:C_0402_1005Metric, F.Cu at (158.4, 21.0)
- added C129: 0.1uF, Capacitor_SMD:C_0603_1608Metric, F.Cu at (134.3, 24.0)
- added C130: 0.1uF, Capacitor_SMD:C_0603_1608Metric, F.Cu at (134.3, 26.5)
- added C131: 100pF, Capacitor_SMD:C_0603_1608Metric, F.Cu at (134.3, 29.0)
- added C132: 1nF, Capacitor_SMD:C_0402_1005Metric, F.Cu at (158.4, 23.0)
- added C133: 1nF, Capacitor_SMD:C_0402_1005Metric, F.Cu at (161.2, 11.2)
- added C134: 0.1uF, Capacitor_SMD:C_0603_1608Metric, F.Cu at (134.3, 31.5)
- added C135: 0.1uF, Capacitor_SMD:C_0603_1608Metric, F.Cu at (134.3, 34.0)
- added C136: 100pF, Capacitor_SMD:C_0603_1608Metric, F.Cu at (134.3, 36.5)
- added C137: 10uF, Capacitor_SMD:C_0603_1608Metric, F.Cu at (134.3, 39.0)
- added C138: 0.1uF, Capacitor_SMD:C_0603_1608Metric, F.Cu at (134.3, 41.5)
- added C139: 10uF, Capacitor_SMD:C_0603_1608Metric, F.Cu at (134.3, 44.0)
- added C140: 10uF, Capacitor_SMD:C_0603_1608Metric, F.Cu at (134.3, 46.6)
- added C141: 0.1uF, Capacitor_SMD:C_0603_1608Metric, F.Cu at (134.3, 49.1)
- added C142: 10uF, Capacitor_SMD:C_0603_1608Metric, F.Cu at (138.3, 11.4)
- added C143: 0.1uF, Capacitor_SMD:C_0603_1608Metric, F.Cu at (138.3, 13.9)
- added C144: 10uF, Capacitor_SMD:C_0603_1608Metric, F.Cu at (138.3, 16.4)
- added C145: 10uF, Capacitor_SMD:C_0603_1608Metric, F.Cu at (138.3, 18.9)
- added C146: 0.1uF, Capacitor_SMD:C_0603_1608Metric, F.Cu at (138.3, 21.5)
- added C147: 0.1uF, Capacitor_SMD:C_0603_1608Metric, F.Cu at (138.3, 24.0)
- added C148: 10uF, Capacitor_SMD:C_0603_1608Metric, F.Cu at (138.3, 26.5)
- added C149: 100pF, Capacitor_SMD:C_0603_1608Metric, F.Cu at (138.3, 29.0)
- added C150: 0.1uF, Capacitor_SMD:C_0603_1608Metric, F.Cu at (138.3, 31.5)
- added C151: 0.1uF, Capacitor_SMD:C_0603_1608Metric, F.Cu at (138.3, 34.0)
- added C152: 1nF, Capacitor_SMD:C_0402_1005Metric, F.Cu at (161.2, 13.1)
- added C153: 10uF, Capacitor_SMD:C_0603_1608Metric, F.Cu at (138.3, 36.5)
- added C154: 10uF, Capacitor_SMD:C_0603_1608Metric, F.Cu at (138.3, 39.0)
- added C155: 0.1uF, Capacitor_SMD:C_0603_1608Metric, F.Cu at (138.3, 41.5)
- added C156: 0.1uF, Capacitor_SMD:C_0603_1608Metric, F.Cu at (138.3, 44.0)
- added C157: 10uF, Capacitor_SMD:C_0603_1608Metric, F.Cu at (138.3, 46.6)
- added C158: 22uF, Capacitor_SMD:C_1206_3216Metric, F.Cu at (144.0, 62.0)
- added C159: 1nF, Capacitor_SMD:C_0402_1005Metric, F.Cu at (161.2, 15.1)
- added C160: 1nF, Capacitor_SMD:C_0402_1005Metric, F.Cu at (161.2, 17.1)
- added C161: 100pF, Capacitor_SMD:C_0603_1608Metric, F.Cu at (138.3, 49.1)
- added C162: 1nF, Capacitor_SMD:C_0402_1005Metric, F.Cu at (161.2, 19.0)
- added C163: 0.1uF, Capacitor_SMD:C_0603_1608Metric, F.Cu at (142.3, 11.4)
- added C164: 0.1uF, Capacitor_SMD:C_0603_1608Metric, F.Cu at (142.3, 13.9)
- added C165: 0.1uF, Capacitor_SMD:C_0603_1608Metric, F.Cu at (142.3, 16.4)
- added C166: 0.1uF, Capacitor_SMD:C_0603_1608Metric, F.Cu at (142.3, 18.9)
- added C167: 22uF, Capacitor_SMD:C_1206_3216Metric, F.Cu at (144.0, 65.4)
- added C168: 1nF, Capacitor_SMD:C_0402_1005Metric, F.Cu at (161.2, 21.0)
- added C169: 0.1uF, Capacitor_SMD:C_0603_1608Metric, F.Cu at (142.3, 21.5)
- added C170: 1nF, Capacitor_SMD:C_0402_1005Metric, F.Cu at (161.2, 23.0)
- added C171: 10uF, Capacitor_SMD:C_0603_1608Metric, F.Cu at (142.3, 24.0)
- added C172: 10uF, Capacitor_SMD:C_0603_1608Metric, F.Cu at (142.3, 26.5)
- added C173: 10uF, Capacitor_SMD:C_0603_1608Metric, F.Cu at (142.3, 29.0)
- added C174: 10uF, Capacitor_SMD:C_0603_1608Metric, F.Cu at (142.3, 31.5)
- added J4: Conn_01x04_Pin, Connector_PinHeader_2.54mm:PinHeader_1x04_P2.54mm_Vertical, F.Cu at (165.0, 12.5)
- added J5: Conn_01x04_Pin, Connector_PinHeader_2.54mm:PinHeader_1x04_P2.54mm_Vertical, F.Cu at (169.6, 12.5)
- added J6: Conn_01x04_Pin, Connector_PinHeader_2.54mm:PinHeader_1x04_P2.54mm_Vertical, F.Cu at (174.2, 12.5)
- added J7: Conn_01x02_Pin, Connector_PinHeader_2.54mm:PinHeader_1x02_P2.54mm_Vertical, F.Cu at (179.4, 56.5)
- added J8: USB_B_Micro, Connector_USB:USB_Micro-B_Amphenol_10118193-0001LF_Horizontal, F.Cu at (49.2, 103.5)
- added R53: 0, Resistor_SMD:R_0603_1608Metric, F.Cu at (146.3, 39.0)
- added R54: 0, Resistor_SMD:R_0603_1608Metric, F.Cu at (146.3, 41.5)
- added R55: 0, Resistor_SMD:R_0603_1608Metric, F.Cu at (146.3, 44.0)
- added R56: 0, Resistor_SMD:R_0603_1608Metric, F.Cu at (146.3, 46.6)
- added U7: RP2040, Package_DFN_QFN:QFN-56-1EP_7x7mm_P0.4mm_EP3.2x3.2mm_ThermalVias, F.Cu at (164.2, 68.2)
- added U8: 8M-Q, Package_SO:SOIC-8_5.3x5.3mm_P1.27mm, F.Cu at (153.5, 75.5)
- added Y2: 12M, Crystal:Crystal_SMD_HC49-SD, F.Cu at (137.2, 70.5)
- added Y3: 25M, Crystal:Crystal_SMD_HC49-SD, F.Cu at (137.2, 77.2)
- C85: value 0.1uF -> 22uF; footprint Capacitor_SMD:C_0603_1608Metric -> Capacitor_SMD:C_1206_3216Metric
- C86, C92, C94: value 0.1uF -> 1nF; footprint Capacitor_SMD:C_0603_1608Metric -> Capacitor_SMD:C_0402_1005Metric
- C93: value 10uF -> 100pF
- C95, C97: value 10uF -> 0.1uF
- IC7: value OPA2673IRGVR -> LIF-MD6000-6UMG64I; footprint Package_DFN_QFN:QFN-16-1EP_4x4mm_P0.65mm_EP2.1x2.1mm_ThermalVias -> LIF-MD6000-6UMG64I:BGA64C40P8X8_350X350X100
- J1: value Conn_01x02_Pin -> RJ45; footprint Connector:JWT_A3963_1x02_P3.96mm_Vertical -> Connector_RJ:RJ45_Amphenol_54602-x08_Horizontal
- R38, R48, R49: value 1k -> 0; footprint Resistor_SMD:R_0805_2012Metric -> Resistor_SMD:R_0603_1608Metric
- R39, R40, R43: value 1k -> 27.4; footprint Resistor_SMD:R_0805_2012Metric -> Resistor_SMD:R_0402_1005Metric
- R47: value 1k -> 50; footprint Resistor_SMD:R_0805_2012Metric -> Resistor_SMD:R_0201_0603Metric
- U6: value DSP -> KSZ9031RNXCA; footprint Package_DFN_QFN:VQFN-48-1EP_6x6mm_P0.4mm_EP4.1x4.1mm_ThermalVias -> Package_DFN_QFN:QFN-48-1EP_7x7mm_P0.5mm_EP5.15x5.15mm_ThermalVias
- moved C41 166.7 mm to (152.6, 11.2), turned to 0 degrees
- moved R47 163.3 mm to (175.0, 66.9), turned to 0 degrees
- moved R14 162.6 mm to (146.3, 11.4), turned to 0 degrees
- moved TP1 161.8 mm to (178.5, 64.9)
- moved TP2 161.6 mm to (178.5, 69.5)
- moved C37 159.1 mm to (149.8, 17.1)
- moved J3 157.3 mm to (166.2, 27.4), turned to 0 degrees
- moved C39 155.5 mm to (149.8, 21.0)
- moved C38 155.1 mm to (149.8, 19.0), turned to 0 degrees
- moved C40 155.0 mm to (149.8, 23.0)
- moved Y1 153.9 mm to (175.4, 36.8), turned to 0 degrees
- moved Q6 153.8 mm to (180.9, 11.5), turned to 0 degrees
- moved IC7 153.5 mm to (162.8, 76.2), turned to 0 degrees
- moved R37 152.8 mm to (146.3, 24.0)
- moved C3 150.9 mm to (176.0, 25.5), turned to 0 degrees
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Connections:
- C85 pad 1: GND -> +3V3
- C85 pad 2: Net-(U6-VDDCORE) -> GND
- C86 pad 2: Net-(U6-VDDCORE) -> +3V3
- C87 pad 2: Net-(U6-AVDD) -> Net-(C87-Pad2)
- C88 pad 1: Net-(U6-AVDD) -> Net-(C87-Pad2)
- C89 pad 1: Net-(U6-AVDD) -> Net-(C87-Pad2)
- C90 pad 2: Net-(U6-AVDD) -> Net-(C87-Pad2)
- C91 pad 1: Net-(U6-AVDD) -> Net-(C87-Pad2)
- C92 pad 1: Net-(IC7-+VS) -> +3V3
- C93 pad 1: Net-(IC7-+VS) -> GND
- C93 pad 2: GND -> +3V3
- C94 pad 1: Net-(IC8-+VS) -> +3V3
- C95 pad 1: Net-(IC8-+VS) -> GND
- C95 pad 2: GND -> +3V3
- C96 pad 1: Net-(IC9-+VS) -> +3V3
- C97 pad 1: Net-(IC9-+VS) -> GND
- C97 pad 2: GND -> +3V3
- IC1 pad 24: GND -> Net-(IC1-CSB)
- J1 pad 1: GND -> Net-(U6-TXRXM_D)
- J1 pad 2: +BATT -> Net-(U6-TXRXP_D)
- R37 pad 2: Net-(U6-AVDD) -> Net-(C87-Pad2)
- R38 pad 1: GND -> Net-(U7-GPIO26_ADC0)
- R38 pad 2: Net-(IC7-+VS) -> Net-(IC3-RFOUT/VD)
- R39 pad 1: Net-(IC7-+VS) -> Net-(J8-D+)
- R39 pad 2: +5V -> Net-(U7-USB_DP)
- R40 pad 1: GND -> Net-(J8-D-)
- R40 pad 2: Net-(IC8-+VS) -> Net-(U7-USB_DM)
- R41 pad 1: Net-(IC8-+VS) -> Net-(C121-Pad1)
- R41 pad 2: +5V -> Net-(U7-XOUT)
- R42 pad 1: GND -> Net-(U6-RESET_N)
- R42 pad 2: Net-(IC9-+VS) -> +3V3
- R43 pad 1: Net-(IC9-+VS) -> Net-(U7-GPIO29_ADC3)
- R47 pad 1: Net-(U6-RD6) -> Net-(U7-GPIO29_ADC3)
- R47 pad 2: +5V -> GND
- R48 pad 1: GND -> Net-(U6-AVDDL_PLL)
- R48 pad 2: Net-(U6-RD6) -> Net-(U6-LDO_O)
- R49 pad 1: Net-(U6-RD6) -> Net-(C141-Pad2)
- R49 pad 2: GND -> Net-(U6-AVDDL_PLL)
- U1 pad 10: Net-(U1-D1) -> Net-(IC7-PB29D)
- U1 pad 11: Net-(U1-D2) -> Net-(IC7-PB16D)
- U1 pad 12: Net-(U1-D3) -> Net-(IC7-PB16C)
- U1 pad 13: Net-(U1-D4) -> Net-(IC7-PB12D)
- U1 pad 14: Net-(U1-D5) -> Net-(IC7-PB12C)
- U1 pad 17: Net-(U1-D6) -> Net-(IC7-PB34C)
- U1 pad 18: Net-(U1-D7) -> Net-(IC7-PB34D)
- U1 pad 19: Net-(U1-D8) -> Net-(IC7-PB2C)
- U1 pad 2: Net-(U1-CLK) -> Net-(IC7-PB29B)
- U1 pad 20: Net-(U1-D9_MSB) -> Net-(IC7-PB2D)
- U1 pad 21: Net-(U1-OR) -> Net-(IC7-PB29A)
- U1 pad 9: Net-(U1-D0_LSB) -> Net-(IC7-PB29C)
- U6 pad 1: Net-(U1-CLK) -> Net-(C148-Pad2)
- U6 pad 10: Net-(U1-D4) -> Net-(U6-TXRXP_D)
- U6 pad 11: Net-(U1-D3) -> Net-(U6-TXRXM_D)
- U6 pad 12: Net-(U1-D2) -> Net-(C148-Pad2)
- U6 pad 13: Net-(U1-D1) -> unconnected-(U6-NC-Pad13)
- U6 pad 14: GND -> Net-(C143-Pad2)
- U6 pad 15: +3V3 -> unconnected-(U6-LED2/PHYAD1-Pad15)
- U6 pad 16: Net-(U1-D0_LSB) -> Net-(C155-Pad2)
- U6 pad 17: Net-(IC7-OUT_A) -> unconnected-(U6-LED1/PHAD0/PME_N1-Pad17)
- U6 pad 18: Net-(IC7-OUTB) -> Net-(C143-Pad2)
- U6 pad 19: GND -> Net-(IC7-PB47)
- U6 pad 2: Net-(U1-OR) -> Net-(U6-TXRXP_A)
- U6 pad 20: +3V3 -> Net-(IC7-PB34B)
- U6 pad 21: Net-(IC8-OUT_A) -> Net-(IC7-PB34A)
- U6 pad 22: Net-(IC8-OUTB) -> Net-(IC7-PB12A)
- U6 pad 23: Net-(IC9-OUT_A) -> Net-(C143-Pad2)
- U6 pad 24: Net-(IC9-OUTB) -> Net-(IC7-PB16A)
- U6 pad 25: Net-(IC5-IN-) -> Net-(IC7-PB48)
- U6 pad 26: GND -> Net-(C143-Pad2)
- U6 pad 27: GND -> Net-(IC7-PB38D)
- U6 pad 28: +3V3 -> Net-(IC7-PB6B)
- U6 pad 29: Net-(Q1-G) -> GND
- U6 pad 3: Net-(U1-D9_MSB) -> Net-(U6-TXRXM_A)
- U6 pad 30: Net-(IC1-MUXOUT) -> Net-(C143-Pad2)
- U6 pad 31: Net-(IC1-SDI) -> Net-(IC7-PB6A)
- U6 pad 32: Net-(IC1-SCK) -> Net-(IC7-PB12B)
- U6 pad 33: Net-(Q3-G) -> Net-(IC7-PB16B)
- U6 pad 34: Net-(IC1-CE) -> Net-(C155-Pad2)
- U6 pad 35: GND -> Net-(IC7-PB38C)
- U6 pad 36: +3V3 -> Net-(U6-MDC)
- U6 pad 37: Net-(Q10-G) -> Net-(U6-MDIO)
- U6 pad 38: Net-(Q8-G) -> Net-(U6-INT_N/PME_N2)
- U6 pad 39: +3V3 -> Net-(C143-Pad2)
- U6 pad 4: Net-(U1-D8) -> Net-(C141-Pad2)
- U6 pad 40: +3.3VADC -> Net-(C155-Pad2)
- U6 pad 41: +3V3 -> Net-(U6-CLK125_NDO/LED_MODE)
- U6 pad 42: Net-(U6-Lx) -> Net-(U6-RESET_N)
- U6 pad 43: GND -> Net-(U6-LDO_O)
- U6 pad 44: Net-(U6-VDDCORE) -> Net-(U6-AVDDL_PLL)
- U6 pad 45: GND -> Net-(U6-XO)
- U6 pad 46: +3V3 -> Net-(U6-XI)
- U6 pad 47: Net-(U6-RD6) -> unconnected-(U6-NC-Pad47)
- U6 pad 48: unconnected-(U6-~{MCLR}-Pad48) -> GND
- U6 pad 5: Net-(U1-D7) -> Net-(U6-TXRXP_B)
- U6 pad 6: GND -> Net-(U6-TXRXM_B)
- U6 pad 7: Net-(U6-AVDD) -> Net-(U6-TXRXP_C)
- U6 pad 8: Net-(U1-D6) -> Net-(U6-TXRXM_C)
- U6 pad 9: Net-(U1-D5) -> Net-(C141-Pad2)
Routing:
- net +3V3: track 316.4 -> 0.00 mm, vias 49 -> 0
- net GND: track 292.5 -> 0.00 mm, vias 417 -> 0
- net +5V: track 151.9 -> 0.00 mm, vias 12 -> 0
- net +3.3VADC: track 113.1 -> 0.00 mm, vias 12 -> 0
- net Net-(D1-A): track 102.1 -> 0.00 mm, vias 6 -> 0
- net Net-(IC7-+VS): track 65.6 -> 0.00 mm, vias 8 -> 0
- net Net-(IC1-CE): track 57.5 -> 0.00 mm, vias 20 -> 0
- net Net-(Q8-G): track 53.7 -> 0.00 mm, vias 14 -> 0
- net Net-(Q1-G): track 52.7 -> 0.00 mm, vias 12 -> 0
- net Net-(IC9-+VS): track 52.6 -> 0.00 mm, vias 8 -> 0
- net Net-(Q3-G): track 52.1 -> 0.00 mm, vias 16 -> 0
- net Net-(IC1-MUXOUT): track 46.6 -> 0.00 mm, vias 12 -> 0
- net Net-(IC1-SCK): track 46.6 -> 0.00 mm, vias 12 -> 0
- net Net-(IC7-OUTB): track 46.4 -> 0.00 mm, vias 6 -> 0
- net +BATT: track 46.0 -> 0.00 mm
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- removed copper zone on In1.Cu, net GND
- removed copper zone on In2.Cu, net GND
Other:
- board size 120 x 110 mm -> 95 x 95 mm
- rule pad_to_mask_clearance: 0 -> 0.01
