File: Wideband-Test-V1.kicad_sch (KiCad schematic)
At the start: 216 parts, among them IC1 LMX2592RHAT, IC2 BU7205HFV-TR, IC3 GRF3042, IC4 OPA2673IRGVR, IC5 BU7205HFV-TR, IC6 BU7205HFV-TR, IC7 OPA2673IRGVR, IC8 OPA2673IRGVR, IC9 OPA2673IRGVR, J1 Conn_01x02_Pin, J2 Conn_01x02_Pin, J3 Conn_01x04_Pin, P1 USB_C_Plug, Q1 MMBFJ113, Q10 MMBFJ113, Q11 MMBFJ113, Q12 BFP840ESD, Q13 BFP840ESD, Q14 BFP840ESD, Q15 BFP840ESD, Q16 BFP840ESD, Q2 MMBFJ113, Q3 MMBFJ113, Q4 MMBFJ113, Q5 MMBFJ113, Q6 MMBFJ113, Q7 BFP840ESD, Q8 MMBFJ113, Q9 MMBFJ113, T1 CX2041NLT, U1 AD9215BCPZ-105, U2 BGA614H6327XTSA1, U3 LD1117V-3V3, U4 BGA614H6327XTSA1, U5 AP7381-50SA-7, U6 DSP, Y1 Crystal_GND24

Commit message: 1 and a u-turn in hardware
Parts:
- removed C85, C86, C92, C94, C96: 0.1uF, Capacitor_SMD:C_0603_1608Metric, symbol Device:C_Small
- removed C93, C95, C97: 10uF, Capacitor_SMD:C_0603_1608Metric, symbol Device:C_Small
- removed D1, D10, D11, D12, D13, D2, D3, D4, D5, D6, D7, D8, D9: MMBZ15VAL215, Package_TO_SOT_SMD:SOT-323_SC-70, symbol Power_Protection:SP0502BAJT
- removed IC7, IC8, IC9: OPA2673IRGVR, Package_DFN_QFN:QFN-16-1EP_4x4mm_P0.65mm_EP2.1x2.1mm_ThermalVias, symbol OPA2673IRGVR:OPA2673IRGVR
- removed J1: Conn_01x02_Pin, Connector:JWT_A3963_1x02_P3.96mm_Vertical, symbol Connector:Conn_01x02_Pin
- removed L2: 10u, Inductor_SMD:L_0603_1608Metric, symbol Device:L_Small
- removed P1: USB_C_Plug, Connector_USB:USB_C_Receptacle_Molex_105450-0101, symbol Connector:USB_C_Plug
- removed R38, R39, R40, R41, R42, R43, R47, R48, R49: 1k, Resistor_SMD:R_0805_2012Metric, symbol Device:R_Small
- removed U6: DSP, Package_DFN_QFN:VQFN-48-1EP_6x6mm_P0.4mm_EP4.1x4.1mm_ThermalVias, symbol DSP_Microchip_DSPIC33:dsPIC33AK256MC505
- added IC7: LIF-MD6000-6UMG64I, LIF-MD6000-6UMG64I:BGA64C40P8X8_350X350X100, symbol LIF-MD6000-6UMG64I:LIF-MD6000-6UMG64I
- added J1: RJ45, Connector_RJ:RJ45_Amphenol_54602-x08_Horizontal, symbol Connector:RJ45
- added U6: KSZ9031RNXCA, Package_DFN_QFN:QFN-48-1EP_7x7mm_P0.5mm_EP5.15x5.15mm, symbol Interface_Ethernet:KSZ9031RNXCA
- added U7: RP2040, Package_DFN_QFN:QFN-56-1EP_7x7mm_P0.4mm_EP3.2x3.2mm, symbol MCU_RaspberryPi:RP2040
- added U8: 8M-Q, Package_SO:SOIC-8_5.3x5.3mm_P1.27mm, symbol IS25LPxxD:IS25LP080D
- added Y2: Crystal_Small, Crystal:Crystal_SMD_HC49-SD, symbol Device:Crystal_Small
Connections:
- net GND: no longer IC1.24 (CSB)
- net at U1.10 (D1): now also IC7.H4 (PB29D)
- net at U1.11 (D2): now also IC7.H5 (PB16D)
- net at U1.12 (D3): now also IC7.H6 (PB16C)
- net at U1.13 (D4): now also IC7.H7 (PB12D)
- net at U1.14 (D5): now also IC7.H8 (PB12C)
- net at U1.17 (D6): now also IC7.H2 (PB34C)
- net at U1.18 (D7): now also IC7.H1 (PB34D)
- net at U1.19 (D8): now also IC7.G8 (PB2C)
- net at U1.2 (CLK): now also IC7.G5 (PB29B)
- net at U1.20 (D9_MSB): now also IC7.G7 (PB2D)
- net at U1.21 (OR): now also IC7.G6 (PB29A)
- net at U1.9 (D0_LSB): now also IC7.H3 (PB29C)
- new net: J1.1, U6.11 (TXRXM_D)
- new net: J1.2, U6.10 (TXRXP_D)
- new net: J1.3, U6.6 (TXRXM_B)
- new net: J1.4, U6.8 (TXRXM_C)
- new net: J1.5, U6.7 (TXRXP_C)
- new net: J1.6, U6.5 (TXRXP_B)
- new net: J1.7, U6.3 (TXRXM_A)
- new net: J1.8, U6.2 (TXRXP_A)
- new net: U7.56 (QSPI_SS), U8.1 (CE)
- new net: U7.55 (QSPI_SD1), U8.2 (IO1(SO))
- new net: U7.54 (QSPI_SD2), U8.3 (IO2(WP))
- new net: U7.53 (QSPI_SD0), U8.5 (IO0(SI))
- new net: U7.52 (QSPI_SCLK), U8.6 (SCK)
- new net: U7.51 (QSPI_SD3), U8.7 (IO3(RESET))
- new net: IC7.C3 (PB47), U6.19 (TXD0)
- new net: IC7.D1 (PB34B), U6.20 (TXD1)
- new net: IC7.D2 (PB34A), U6.21 (TXD2)
- new net: IC7.D8 (PB12A), U6.22 (TXD3)
- new net: IC7.D7 (PB16A), U6.24 (GTX_CLK)
- new net: IC7.E3 (PB48), U6.25 (TX_EN)
- new net: IC7.G1 (PB38D), U6.27 (RXD3/MODE3)
- new net: IC7.F8 (PB6B), U6.28 (RXD2/MODE2)
- new net: IC7.F7 (PB6A), U6.31 (RXD1/MODE1)
- new net: IC7.E8 (PB12B), U6.32 (RXD0/MODE0)
- new net: IC7.E7 (PB16B), U6.33 (RX_DV/CLK125_EN)
- new net: IC7.G2 (PB38C), U6.35 (RX_CLK/PHYAD2)
- new net: U7.1 (IOVDD), U7.10 (IOVDD), U7.22 (IOVDD), U7.33 (IOVDD), U7.42 (IOVDD), U7.49 (IOVDD)
- new net: U7.23 (DVDD), U7.50 (DVDD)
Other:
- moved on the sheet: C42, C43, C44, C51, C52, C53, C54, C55, C56, C57, C58, C59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

Commit message: 1.x
Parts:
- added C103, C108, C111, C112, C114, C115, C116, C117, C129, C130, C134, C135, C138, C141, C143, C146, C147, C150, C151, C155, C156, C163, C164, C165, C166, C169, C95, C96, C97: 0.1uF, Capacitor_SMD:C_0603_1608Metric, symbol Device:C_Small
- added C104, C110, C113, C125, C126, C137, C139, C140, C142, C144, C145, C148, C153, C154, C157, C171, C172, C173, C174: 10uF, Capacitor_SMD:C_0603_1608Metric, symbol Device:C_Small
- added C105, C107, C158, C167, C85: 22uF, Capacitor_SMD:C_1206_3216Metric, symbol Device:C_Small
- added C106, C109, C118, C119, C127, C128, C132, C133, C152, C159, C160, C162, C168, C170, C86, C92, C94: 1nF, Capacitor_SMD:C_0402_1005Metric, symbol Device:C
- added C120, C131, C136, C149, C161, C93: 100pF, Capacitor_SMD:C_0603_1608Metric, symbol Device:C
- added C121, C122, C123, C124: 30pF, Capacitor_SMD:C_0603_1608Metric, symbol Device:C
- added J4, J5, J6: Conn_01x04_Pin, Connector_PinHeader_2.54mm:PinHeader_1x04_P2.54mm_Vertical, symbol Connector:Conn_01x04_Pin
- added J7: Conn_01x02_Pin, Connector_PinHeader_2.54mm:PinHeader_1x02_P2.54mm_Vertical, symbol Connector:Conn_01x02_Pin
- added J8: USB_B_Micro, Connector_USB:USB_Micro-B_Amphenol_10118193-0001LF_Horizontal, symbol Connector:USB_B_Micro
- added R38, R48, R49, R53, R54, R55, R56: 0, Resistor_SMD:R_0603_1608Metric, symbol Device:R_Small
- added R39, R40, R43: 27.4, Resistor_SMD:R_0402_1005Metric, symbol Device:R_Small
- added R41, R42: 1k, Resistor_SMD:R_0805_2012Metric, symbol Device:R_Small
- added R47: 50, Resistor_SMD:R_0201_0603Metric, symbol Device:R_Small
- added Y3: 25M, Crystal:Crystal_SMD_HC49-SD, symbol Device:Crystal_Small
- U6: footprint Package_DFN_QFN:QFN-48-1EP_7x7mm_P0.5mm_EP5.15x5.15mm -> Package_DFN_QFN:QFN-48-1EP_7x7mm_P0.5mm_EP5.15x5.15mm_ThermalVias
- U7: footprint Package_DFN_QFN:QFN-56-1EP_7x7mm_P0.4mm_EP3.2x3.2mm -> Package_DFN_QFN:QFN-56-1EP_7x7mm_P0.4mm_EP3.2x3.2mm_ThermalVias
- Y2: value Crystal_Small -> 12M
Connections:
- net +3.3VADC: now also U7.39 (GPIO27_ADC1)
- net +3V3: now also U7.1 (IOVDD), U7.10 (IOVDD), U7.22 (IOVDD), U7.33 (IOVDD), U7.40 (GPIO28_ADC2), U7.42 (IOVDD), U7.43 (ADC_AVDD), U7.44 (VREG_IN), U7.48 (USB_VDD), U7.49 (IOVDD), U8.8 (VCC), C103.1, C104.2, C105.1, C106.1, C107.2, C108.2, C109.1, C110.1, C111.2, C112.2, C85.1, C86.2, C92.1, C93.2, C94.1, C95.2, C96.1, C97.2, J5.1 (Pin_1), R42.2, R54.2, R55.2, R56.1
- net +5V: now also J8.1 (VBUS), R43.2
- net GND: now also IC7.C6 (GNDA_DPHYX), IC7.D4 (GND_1), IC7.E5 (GND_2), IC7.F5 (GND_3), U6.29 (VSS), U6.48 (ISET), U6.49 (PAD_GND), U7.57 (GND), U8.4 (GND), C103.2, C104.1, C105.2, C106.2, C107.1, C108.1, C109.2, C110.2, C111.1, C112.1, C113.1, C114.1, C115.1, C116.1, C117.1, C118.1, C119.1, C120.1, C121.2, C122.2, C123.2, C124.2, C125.1, C126.1, C127.1, C128.1, C129.1, C130.1, C131.1, C132.1, C133.1, C134.1, C135.1, C136.1, C137.1, C138.1, C139.1, C140.1, C141.1, C142.1, C143.1, C144.1, C145.1, C146.1, C147.1, C148.1, C149.1, C150.1, C151.1, C152.1, C153.2, C154.2, C155.1, C156.1, C157.1, C158.2, C159.1, C160.2, C161.1, C162.2, C163.1, C164.2, C165.1, C166.2, C167.2, C168.2, C169.1, C170.2, C171.2, C172.1, C173.2, C174.1, C85.2, C86.1, C92.2, C93.1, C94.2, C95.1, C96.2, C97.1, J6.1 (Pin_1), J8.5 (GND), J8.6 (Shield), R47.2; no longer AE3.2 (PCB_Trace)
- net at Q10.3 (G), Q11.3 (G): now also U7.17 (GPIO14)
- net at Q3.3 (G), Q4.3 (G): now also U7.16 (GPIO13)
- net at IC1.1 (CE): now also U7.2 (GPIO0)
- net at IC1.16 (SCK): now also U7.4 (GPIO2)
- net at IC1.17 (SDI): now also U7.5 (GPIO3)
- net at IC1.20 (MUXOUT): now also U7.11 (GPIO8)
- net at IC1.24 (CSB): now also U7.3 (GPIO1)
- net at Q8.3 (G), Q9.3 (G): now also U7.18 (GPIO15)
- net at C102.1, IC3.4 (RFOUT/VD), L1.2: now also R38.2
- net at IC5.3 (IN-), IC6.1 (IN+): now also U7.8 (GPIO6)
- net at U6.1 (AVDDH): now also U6.12 (AVDDH), C148.2, C149.2, C150.2, C151.2, C152.2, C153.1, C154.1, R54.1
- net at U6.14 (DVDDL): now also U6.18 (DVDDL), U6.23 (DVDDL), U6.26 (DVDDL), U6.30 (DVDDL), U6.39 (DVDDL), C143.2, C144.2, C147.2, R53.1
- net at U6.16 (DVDDH): now also U6.34 (DVDDH), U6.40 (DVDDH), C155.2, C156.2, C157.2, R55.1
- net at U6.36 (MDC): now also U7.34 (GPIO22)
- net at U6.37 (MDIO): now also U7.35 (GPIO23)
- net at U6.38 (INT_N/PME_N2): now also U7.30 (GPIO19)
- net at U6.4 (AVDDL): now also U6.9 (AVDDL), C141.2, C142.2, C145.2, C146.2, R49.1, R53.2
- net at U6.41 (CLK125_NDO/LED_MODE): now also U7.29 (GPIO18)
- net at U6.42 (RESET_N): now also U7.28 (GPIO17), C125.2, R42.1
- net at U6.43 (LDO_O): now also C126.2, C127.2, C128.2, C129.2, C130.2, C131.2, C132.2, C133.2, C134.2, C135.2, C136.2, C137.2, C139.2, R48.2
- net at U6.44 (AVDDL_PLL): now also C138.2, C140.2, R48.1, R49.2
- net at U6.45 (XO): now also C123.1, Y3.2
- net at U6.46 (XI): now also C124.1, Y3.1
- net at U7.12 (GPIO9): now also IC7.D3 (PB52), J6.2 (Pin_2)
- net at U7.13 (GPIO10): now also IC7.F1 (PB53), J5.3 (Pin_3)
- net at U7.14 (GPIO11): now also IC7.F2 (PB50), J6.3 (Pin_3)
- net at U7.15 (GPIO12): now also IC7.E1 (PB51), J5.2 (Pin_2)
- net at U7.19 (TESTEN): now also J4.4 (Pin_4)
- net at U7.20 (XIN): now also Y2.2, C122.1
- net at U7.21 (XOUT): now also R41.2
- net at U7.23 (DVDD), U7.50 (DVDD): now also U7.45 (VREG_VOUT), C113.2, C114.2, C115.2, C116.2, C117.2, C118.2, C119.2, C120.2
- net at U7.24 (SWCLK): now also J4.1 (Pin_1)
- net at U7.25 (SWD): now also J4.2 (Pin_2)
- net at U7.26 (RUN): now also J4.3 (Pin_3)
- net at U7.27 (GPIO16): now also IC7.G3 (PB49), U7.7 (GPIO5), J6.4 (Pin_4)
- net at U7.31 (GPIO20): now also U7.32 (GPIO21)
- net at U7.36 (GPIO24): now also J7.2 (Pin_2)
- net at U7.37 (GPIO25): now also J7.1 (Pin_1)
- net at U7.38 (GPIO26_ADC0): now also R38.1
- net at U7.41 (GPIO29_ADC3): now also R43.1, R47.1
- net at U7.46 (USB_DM): now also R40.2
- net at U7.47 (USB_DP): now also R39.2
- net at U7.6 (GPIO4): now also IC7.E2 (CRESET_B), J5.4 (Pin_4)
- net at U7.9 (GPIO7): now also Q1.3 (G), Q2.3 (G)
- net VCC: now reaches IC7.C4 (VCCPLL_DPHYX)
- net VCC: now also IC7.C5 (VCCA_DPHYX), IC7.D5 (VCC_1), IC7.D6 (VCCAUX), IC7.E4 (VCC_2), IC7.E6 (VCCIO2_1), IC7.F3 (VCCIO0), IC7.F4 (VCCIO1), IC7.F6 (VCCIO2_2), IC7.G4 (VCCGPLL), C158.1, C159.2, C160.1, C161.2, C162.1, C163.2, C164.1, C165.2, C166.1, C167.1, C168.1, C169.2, C170.1, C171.1, C172.2, C173.1, C174.2, R56.2
- net at Y2.1: now also C121.1, R41.1
- new net: J8.2 (D-), R40.1
- new net: J8.3 (D+), R39.1
Other:
- moved on the sheet: C51, C52, C53, C66, C67, C68, C69, R52, U3, U5
