File: hardware/Wideband-Test-V1.kicad_pcb (KiCad board)
At the start: 4 copper layers, 95 x 95 mm, 280 parts, among them IC1 LMX2592RHAT, IC2 BU7205HFV-TR, IC3 GRF3042, IC4 OPA2673IRGVR, IC5 BU7205HFV-TR, IC6 BU7205HFV-TR, IC7 LIF-MD6000-6UMG64I, J1 RJ45, J2 Conn_01x02_Pin, J3 Conn_01x04_Pin, J4 Conn_01x04_Pin, J5 Conn_01x04_Pin, J6 Conn_01x04_Pin, J7 Conn_01x02_Pin, J8 USB_B_Micro, Q1 MMBFJ113, Q10 MMBFJ113, Q11 MMBFJ113, Q12 BFP840ESD, Q13 BFP840ESD, Q14 BFP840ESD, Q15 BFP840ESD, Q16 BFP840ESD, Q2 MMBFJ113, Q3 MMBFJ113, Q4 MMBFJ113, Q5 MMBFJ113, Q6 MMBFJ113, Q7 BFP840ESD, Q8 MMBFJ113, Q9 MMBFJ113, U1 AD9215BCPZ-105, U2 BGA614H6327XTSA1, U3 LD1117V-3V3, U4 BGA614H6327XTSA1, U5 AP7381-50SA-7, U6 KSZ9031RNXCA, U7 RP2040, U8 8M-Q, Y1 Crystal_GND24, Y2 12M, Y3 25M

Commit message: hardwares
Parts:
- removed J7: Conn_01x02_Pin, Connector_PinHeader_2.54mm:PinHeader_1x02_P2.54mm_Vertical
- removed Q10, Q11, Q8, Q9: MMBFJ113, Package_DFN_QFN:Diodes_DFN1006-3
- added AE1: Antenna_Chip, Connector_Coaxial:SMA_Molex_73251-2200_Horizontal, F.Cu at (115.1, 34.3)
- added AE2: Antenna_Chip, Connector_Coaxial:SMA_Molex_73251-2200_Horizontal, F.Cu at (115.2, 25.1)
- added AE3: Antenna_Chip, Connector_Coaxial:SMA_Molex_73251-2200_Horizontal, F.Cu at (115.2, 16.1)
- added T1: CX2041NLT, Filter:Filter_SAW-6_3.8x3.8mm, F.Cu at (69.3, 13.4)
- added U10: BGS12WN6E6327, Package_LGA:Infineon_PG-TSNP-6-10_0.7x1.1mm_0.7x1.1mm_P0.4mm, F.Cu at (92.2, 15.3)
- added U11: BGS12WN6E6327, Package_LGA:Infineon_PG-TSNP-6-10_0.7x1.1mm_0.7x1.1mm_P0.4mm, F.Cu at (95.4, 22.6)
- added U12: BGS12WN6E6327, Package_LGA:Infineon_PG-TSNP-6-10_0.7x1.1mm_0.7x1.1mm_P0.4mm, F.Cu at (97.0, 22.6)
- added U13: BGS12WN6E6327, Package_LGA:Infineon_PG-TSNP-6-10_0.7x1.1mm_0.7x1.1mm_P0.4mm, F.Cu at (57.8, 14.9)
- added U14: BGS12WN6E6327, Package_LGA:Infineon_PG-TSNP-6-10_0.7x1.1mm_0.7x1.1mm_P0.4mm, F.Cu at (58.0, 13.5)
- added U9: BGS12WN6E6327, Package_LGA:Infineon_PG-TSNP-6-10_0.7x1.1mm_0.7x1.1mm_P0.4mm, F.Cu at (89.0, 15.3)
- TR1, TR2, TR3: footprint Package_DIP:SMDIP-6_W7.62mm -> MABA-011108:MABA011108
- moved U5 171.5 mm to (11.6, 36.6)
- moved U3 165.8 mm to (2.71, 3.60)
- moved J2 160.5 mm to (2.54, 36.7)
- moved Y3 143.1 mm to (9.19, 13.2)
- moved J6 143.0 mm to (33.5, 38.2), turned to 90 degrees
- moved U6 142.9 mm to (25.4, 25.1)
- moved TP1 140.5 mm to (52.9, 1.84), turned to 90 degrees
- moved J3 140.1 mm to (28.2, 3.03)
- moved TP2 138.6 mm to (57.5, 1.84), turned to 90 degrees
- moved J5 137.9 mm to (33.4, 34.7), turned to 90 degrees
- moved U1 135.0 mm to (52.6, 14.6), turned to -90 degrees
- moved U8 134.0 mm to (25.5, 35.9)
- moved IC7 131.9 mm to (42.9, 21.0), turned to 180 degrees
- moved R19 126.6 mm to (56.5, 14.5), turned to 180 degrees
- moved R18 126.2 mm to (56.5, 13.8)
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Connections:
- C6 pad 2: Net-(IC1-GND_2) -> GND
- IC1 pad 4: Net-(IC1-GND_2) -> GND
- IC1 pad 6: Net-(IC1-GND_2) -> GND
- U2 pad 3: INAMP+ -> Net-(U13-RFIN)
- U4 pad 3: INAMP- -> Net-(U14-RFIN)
- U7 pad 31: Net-(U7-GPIO20) -> ANT3+
- U7 pad 32: Net-(U7-GPIO20) -> ANT3-
- U7 pad 36: Net-(J7-Pin_2) -> unconnected-(U7-GPIO24-Pad36)
Routing:
- net TRANS-: track 0.00 -> 88.1 mm, vias 0 -> 12
- net TRANS+: track 0.00 -> 86.1 mm, vias 0 -> 11
- net GND: track 0.00 -> 82.9 mm, vias 0 -> 17
- net Net-(IC4-+IN_B): track 0.00 -> 72.0 mm, vias 0 -> 5
- net Net-(U14-RFIN): track 0.00 -> 42.5 mm, vias 0 -> 5
- net Net-(Q6-S): track 0.00 -> 39.9 mm, vias 0 -> 12
- net +3V3: track 0.00 -> 37.7 mm, vias 0 -> 3
- net ANT123+: track 0.00 -> 32.5 mm
- net ANT123-: track 0.00 -> 29.5 mm, vias 0 -> 5
- net ANT3+: track 0.00 -> 29.3 mm
- net OPA+: track 0.00 -> 25.8 mm, vias 0 -> 6
- net Net-(IC3-RFIN): track 0.00 -> 24.7 mm, vias 0 -> 2
- net Net-(IC7-PB29C): track 0.00 -> 24.1 mm
- net Net-(IC4--IN_A): track 0.00 -> 24.0 mm, vias 0 -> 2
- net Net-(IC7-PB34D): track 0.00 -> 21.1 mm
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- added copper zone on F.Cu, net GND
- added copper zone on In1.Cu, net GND
Other:
- board size 95 x 95 mm -> 120 x 40 mm

Commit message: Address issue 12 FFT receive path blockers
Parts:
- moved R42 179.8 mm to (7.17, 7.06)
- moved C152 175.6 mm to (12.8, 7.56), turned to 180 degrees
- moved R54 168.1 mm to (6.96, 10.3)
- moved C133 165.6 mm to (23.4, 18.3), turned to 90 degrees
- moved C148 164.0 mm to (1.71, 9.28), turned to 90 degrees
- moved C145 163.8 mm to (1.66, 12.3), turned to -90 degrees
- moved C149 161.9 mm to (3.96, 8.79), turned to 180 degrees
- moved C146 161.5 mm to (3.94, 10.3), turned to 180 degrees
- moved C127 161.3 mm to (24.4, 18.3), turned to 90 degrees
- moved C128 160.3 mm to (25.3, 18.3), turned to 90 degrees
- moved C124 159.9 mm to (1.67, 15.3), turned to -90 degrees
- moved C132 159.3 mm to (26.3, 18.3), turned to 90 degrees
- moved C150 159.1 mm to (6.96, 8.80), turned to 180 degrees
- moved C153 157.4 mm to (9.21, 9.54), turned to 90 degrees
- moved C120 156.6 mm to (3.96, 7.29), turned to 180 degrees
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Connections:
- C155 pad 2: Net-(C155-Pad2) -> Net-(U7-VREG_VOUT)
- C156 pad 2: Net-(C155-Pad2) -> Net-(U7-VREG_VOUT)
- C157 pad 2: Net-(C155-Pad2) -> Net-(U7-VREG_VOUT)
- R55 pad 1: Net-(C155-Pad2) -> Net-(U7-VREG_VOUT)
- U6 pad 16: Net-(C155-Pad2) -> Net-(U7-VREG_VOUT)
- U6 pad 34: Net-(C155-Pad2) -> Net-(U7-VREG_VOUT)
- U6 pad 40: Net-(C155-Pad2) -> Net-(U7-VREG_VOUT)
Routing:
- net Net-(U5-GND): track 0.00 -> 9.28 mm
- net +5V: track 0.00 -> 8.46 mm
- net +BATT: track 0.00 -> 6.68 mm
- net Net-(J8-D-): track 0.00 -> 1.80 mm
- net Net-(J8-D+): track 0.00 -> 1.65 mm
