File: hardware/v2/sheets/01_power.kicad_sch (KiCad schematic)
At the start: 27 parts, among them J1 5V_INPUT_ONLY, U1 TLV62569DBVR, U2 TLV62569DBVR, U3 TLV75525PDBVR, U4 TLV76733DRVR

Commit message: fix(hardware): use project-local 0805 inductor footprint [skip ci]
Parts:
- FB1, L1, L2: footprint Inductor_SMD:L_0805_2012Metric_Pad1.15x1.40mm_HandSolder -> CodeSDR:Inductor_0805_HandSolder
Changed lines of the file:
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@@
 			)
 		)
-		(property "Footprint" "Inductor_SMD:L_0805_2012Metric_Pad1.15x1.40mm_HandSolder"
+		(property "Footprint" "CodeSDR:Inductor_0805_HandSolder"
 			(at 398.272 90.17 90)
 			(effects
@@
 			)
 		)
-		(property "Footprint" "Inductor_SMD:L_0805_2012Metric_Pad1.15x1.40mm_HandSolder"
+		(property "Footprint" "CodeSDR:Inductor_0805_HandSolder"
 			(at 69.85 142.24 0.0000)
 			(effects
@@
 			)
 		)
-		(property "Footprint" "Inductor_SMD:L_0805_2012Metric_Pad1.15x1.40mm_HandSolder"
+		(property "Footprint" "CodeSDR:Inductor_0805_HandSolder"
 			(at 69.85 194.31 0.0000)
 			(effects

Commit message: hardware: checkpoint corrected V2 routing at 108 opens
Parts:
- added C340, C341, C342, C343, C344, C347: 100nF, Capacitor_SMD:C_0402_1005Metric, symbol Device:C_Small
- added C345: 20nF_C0G_5%, Capacitor_SMD:C_0805_2012Metric, symbol Device:C_Small
- added C346: 47uF_10V_X7R, Capacitor_SMD:C_1210_3225Metric, symbol Device:C_Small
- added C348: 10nF, Capacitor_SMD:C_0402_1005Metric, symbol Device:C_Small
- added R154: 30.3k_0.1%, Resistor_SMD:R_0402_1005Metric, symbol Device:R_Small
- added R155: 10k_0.1%, Resistor_SMD:R_0402_1005Metric, symbol Device:R_Small
- added R157, R159: 120k_1%, Resistor_SMD:R_0402_1005Metric, symbol Device:R_Small
- added R158: 100k_1%, Resistor_SMD:R_0402_1005Metric, symbol Device:R_Small
- added U5, U6, U7: TPS389033DSER, Package_SON:WSON-6_1.5x1.5mm_P0.5mm, symbol CodeSDR:TPS389033DSER
- added U8, U9: TPS389012DSER, Package_SON:WSON-6_1.5x1.5mm_P0.5mm, symbol CodeSDR:TPS389012DSER
- C11: value 4.7uF -> 22uF_10V_X7R; footprint Capacitor_SMD:C_0805_2012Metric -> Capacitor_SMD:C_1206_3216Metric
- C12: value 4.7uF -> 47uF_10V_X7R; footprint Capacitor_SMD:C_0805_2012Metric -> Capacitor_SMD:C_1210_3225Metric
- R1: value 453k_1% -> 453k_0.1%
- R2, R4: value 100k_1% -> 100k_0.1%
- R3: value 100k_1% -> 101k_0.1%
- U4: value TLV76733DRVR -> TPS7A8300ARGWT; footprint Package_SON:WSON-6-1EP_2x2mm_P0.65mm_EP1x1.6mm_ThermalVias -> Package_DFN_QFN:Texas_RGW0020A_VQFN-20-1EP_5x5mm_P0.65mm_EP3.15x3.15mm_ThermalVias; symbol CodeSDR:TLV76733DRVR -> CodeSDR:TPS7A8300ARGWT
Connections:
- net +3V3_ANA: now also U4.19 (OUT), U4.20 (OUT), C346.1, C348.1, R154.1; no longer U4.2 (SNS)
- net +3V3_DIG: now also C340.1, C341.1, C342.1, C343.1, C344.1, R157.1, R159.1, U5.3 (MR_N), U5.4 (VDD), U6.3 (MR_N), U6.4 (VDD), U7.3 (MR_N), U7.4 (VDD), U8.3 (MR_N), U8.4 (VDD), U9.3 (MR_N), U9.4 (VDD); no longer U3.3 (EN)
- net GND: now also U4.12 (BIAS), U4.18 (GND), U4.21 (EP), U4.8 (GND), C340.2, C341.2, C342.2, C343.2, C344.2, C345.2, C346.2, C347.2, R155.2, R158.2, U5.2 (GND), U6.2 (GND), U7.2 (GND), U8.2 (GND), U9.2 (GND); no longer U4.3 (GND), U4.5 (GND), U4.7 (EP)
- net VIN_FUSED: now also U4.14 (EN), U4.15 (IN), U4.16 (IN), U4.17 (IN); no longer U2.1 (EN), U4.4 (EN), U4.6 (IN)
- new net ANA_NR_SS: C347.1, U4.13 (NR_SS)
- new net AUX_EN: R159.2, U3.3 (EN), U8.6 (RESET_N)
- new net CORE_EN: R157.2, R158.1, U2.1 (EN), U5.6 (RESET_N), U6.6 (RESET_N), U7.6 (RESET_N)
- new net FB_ANA: C348.2, R154.2, R155.1, U4.3 (FB)
- new net FPGA_VCCIO0_3V3: U5.1 (SENSE)
- new net FPGA_VCCIO1_3V3: U6.1 (SENSE)
- new net FPGA_VCCIO2_3V3: U7.1 (SENSE)
- new net FPGA_VCC_1V2: U8.1 (SENSE)
- new net PHY_AVDDL_1V2: U9.1 (SENSE)
- new net PHY_RESET_CT: C345.1, U9.5 (CT)
- new net PHY_RESET_N: U9.6 (RESET_N)
- no-connect marks 1 -> 13
