File: hardware/v2/sheets/02_controller.kicad_sch (KiCad schematic)
At the start: 27 parts, among them J10 USB_B_Micro, J11 Cortex_SWD_10pin, SW1 BOOTSEL, SW2 RESET, U10 RP2040, U11 W25Q16JVSSIQ, U12 USBLC6-2SC6, Y10 ABM8-272-T3_12MHz

Commit message: hardware: checkpoint corrected V2 routing at 108 opens
Parts:
- added C330, C331: 100nF, Capacitor_SMD:C_0402_1005Metric, symbol Device:C_Small
- added R150: 1k, Resistor_SMD:R_0201_0603Metric, symbol Device:R_Small
- added R151: 1k, Resistor_SMD:R_0402_1005Metric, symbol Device:R_Small
- C306: value 100nF -> 1uF
- U11: value W25Q16JVSSIQ -> W25Q16JVSNIQ; symbol CodeSDR:W25Q16JVSSIQ -> CodeSDR:W25Q16JVSNIQ
Connections:
- net GND: now also C330.2, C331.2
- net QSPI_SS_N: now also R151.1; no longer SW1.1
- net RP_CORE: now also C330.1, C331.1
- net RP_XOUT: now also R150.2; no longer U10.21 (XOUT)
- new net BOOTSEL_SWITCH: R151.2, SW1.1
- new net RP_XOUT_DRIVE: R150.1, U10.21 (XOUT)
Changed lines of the file:
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@@
 	)
 	(symbol
-		(lib_id "CodeSDR:W25Q16JVSSIQ")
+		(lib_id "CodeSDR:W25Q16JVSNIQ")
 		(at 180.34 90.17 0)
 		(unit 1)
@@
 			)
 		)
-		(property "Value" "W25Q16JVSSIQ"
+		(property "Value" "W25Q16JVSNIQ"
 			(at 180.34 74.93 0.0000)
 			(effects
@@
 			)
 		)
-		(property "Value" "100nF"
+		(property "Value" "1uF"
 			(at 620.014 140.208 0.0000)
 			(effects
@@
 		)
 	)
-	(global_label "RP_XOUT"
+	(global_label "RP_XOUT_DRIVE"
 		(shape bidirectional)
 		(at 46.9900 104.1400 0)
@@
 		)
 	)
-	(global_label "QSPI_SS_N"
+	(global_label "BOOTSEL_SWITCH"
 		(shape bidirectional)
 		(at 284.4800 246.3800 0)
@@
 		)
 	)
+	(symbol (lib_id "Device:R_Small") (at 730.2500 246.3800 0) (unit 1)
+	(exclude_from_sim no) (in_bom yes) (on_board yes)
+	(dnp no)
+	(fields_autoplaced no)
+	(property "Reference" "R150" (at 735.3300 243.8400 0) (effects (font (size 1.27 1.27)) (justify left)))
+	(property "Value" "1k" (at 735.3300 248.9200 0) (effects (font (size 1.27 1.27)) (justify left)))
+	(property "Footprint" "Resistor_SMD:R_0201_0603Metric" (at 735.3300 248.9200 0) (effects (font (size 1.27 1.27)) (justify left) (hide yes)))
+	(property "Datasheet" "" (at 735.3300 248.9200 0) (effects (font (size 1.27 1.27)) (justify left) (hide yes)))
+	(property "Description" "" (at 735.3300 248.9200 0) (effects (font (size 1.27 1.27)) (justify left) (hide yes)))
+	(pin "1")
+	(pin "2")
+	(instances (project "Code-SDR-V2" (path "/b04744a4-fe39-4740-81de-d5e094f9e157/7e81e054-bf24-46f6-919f-d12f5f0aa95a" (reference "R150") (unit 1))))
+)
+	(symbol (lib_id "Device:C_Small") (at 69.8500 298.4500 0) (unit 1)
+	(exclude_from_sim no) (in_bom yes) (on_board yes)
+	(dnp no)
+	(fields_autoplaced no)
+	(property "Reference" "C330" (at 74.9300 295.9100 0) (effects (font (size 1.27 1.27)) (justify left)))
+	(property "Value" "100nF" (at 74.9300 300.9900 0) (effects (font (size 1.27 1.27)) (justify left)))
+	(property "Footprint" "Capacitor_SMD:C_0402_1005Metric" (at 74.9300 300.9900 0) (effects (font (size 1.27 1.27)) (justify left) (hide yes)))
+	(property "Datasheet" "" (at 74.9300 300.9900 0) (effects (font (size 1.27 1.27)) (justify left) (hide yes)))
+	(property "Description" "RP_CORE local bypass" (at 74.9300 300.9900 0) (effects (font (size 1.27 1.27)) (justify left) (hide yes)))
+	(pin "1")
+	(pin "2")
+	(instances (project "Code-SDR-V2" (path "/b04744a4-fe39-4740-81de-d5e094f9e157/7e81e054-bf24-46f6-919f-d12f5f0aa95a" (reference "C330") (unit 1))))
+)
+	(symbol (lib_id "Device:C_Small") (at 180.3400 298.4500 0) (unit 1)
+	(exclude_from_sim no) (in_bom yes) (on_board yes)
+	(dnp no)
+	(fields_autoplaced no)
+	(property "Reference" "C331" (at 185.4200 295.9100 0) (effects (font (size 1.27 1.27)) (justify left)))
+	(property "Value" "100nF" (at 185.4200 300.9900 0) (effects (font (size 1.27 1.27)) (justify left)))
+	(property "Footprint" "Capacitor_SMD:C_0402_1005Metric" (at 185.4200 300.9900 0) (effects (font (size 1.27 1.27)) (justify left) (hide yes)))
+	(property "Datasheet" "" (at 185.4200 300.9900 0) (effects (font (size 1.27 1.27)) (justify left) (hide yes)))
+	(property "Description" "RP_CORE local bypass" (at 185.4200 300.9900 0) (effects (font (size 1.27 1.27)) (justify left) (hide yes)))
+	(pin "1")
+	(pin "2")
+	(instances (project "Code-SDR-V2" (path "/b04744a4-fe39-4740-81de-d5e094f9e157/7e81e054-bf24-46f6-919f-d12f5f0aa95a" (reference "C331") (unit 1))))
+)
+	(symbol (lib_id "Device:R_Small") (at 289.5600 298.4500 0) (unit 1)
+	(exclude_from_sim no) (in_bom yes) (on_board yes)
+	(dnp no)
+	(fields_autoplaced no)
+	(property "Reference" "R151" (at 294.6400 295.9100 0) (effects (font (size 1.27 1.27)) (justify left)))
+	(property "Value" "1k" (at 294.6400 300.9900 0) (effects (font (size 1.27 1.27)) (justify left)))
+	(property "Footprint" "Resistor_SMD:R_0402_1005Metric" (at 294.6400 300.9900 0) (effects (font (size 1.27 1.27)) (justify left) (hide yes)))
+	(property "Datasheet" "" (at 294.6400 300.9900 0) (effects (font (size 1.27 1.27)) (justify left) (hide yes)))
+	(property "Description" "" (at 294.6400 300.9900 0) (effects (font (size 1.27 1.27)) (justify left) (hide yes)))
+	(pin "1")
+	(pin "2")
+	(instances (project "Code-SDR-V2" (path "/b04744a4-fe39-4740-81de-d5e094f9e157/7e81e054-bf24-46f6-919f-d12f5f0aa95a" (reference "R151") (unit 1))))
+)
+	(global_label "RP_XOUT_DRIVE" (shape bidirectional) (at 730.2500 243.8400 0) (fields_autoplaced yes) (effects (font (size 1.27 1.27)) (justify left)) (property "Intersheetrefs" "${INTERSHEET_REFS}" (at 732.7900 243.8400 0) (effects (font (size 1.27 1.27)) (justify left) (hide yes))))
+	(global_label "RP_XOUT" (shape bidirectional) (at 730.2500 248.9200 0) (fields_autoplaced yes) (effects (font (size 1.27 1.27)) (justify left)) (property "Intersheetrefs" "${INTERSHEET_REFS}" (at 732.7900 248.9200 0) (effects (font (size 1.27 1.27)) (justify left) (hide yes))))
+	(global_label "RP_CORE" (shape bidirectional) (at 69.8500 295.9100 0) (fields_autoplaced yes) (effects (font (size 1.27 1.27)) (justify left)) (property "Intersheetrefs" "${INTERSHEET_REFS}" (at 72.3900 295.9100 0) (effects (font (size 1.27 1.27)) (justify left) (hide yes))))
+	(global_label "GND" (shape bidirectional) (at 69.8500 300.9900 0) (fields_autoplaced yes) (effects (font (size 1.27 1.27)) (justify left)) (property "Intersheetrefs" "${INTERSHEET_REFS}" (at 72.3900 300.9900 0) (effects (font (size 1.27 1.27)) (justify left) (hide yes))))
+	(global_label "RP_CORE" (shape bidirectional) (at 180.3400 295.9100 0) (fields_autoplaced yes) (effects (font (size 1.27 1.27)) (justify left)) (property "Intersheetrefs" "${INTERSHEET_REFS}" (at 182.8800 295.9100 0) (effects (font (size 1.27 1.27)) (justify left) (hide yes))))
+	(global_label "GND" (shape bidirectional) (at 180.3400 300.9900 0) (fields_autoplaced yes) (effects (font (size 1.27 1.27)) (justify left)) (property "Intersheetrefs" "${INTERSHEET_REFS}" (at 182.8800 300.9900 0) (effects (font (size 1.27 1.27)) (justify left) (hide yes))))
+	(global_label "QSPI_SS_N" (shape bidirectional) (at 289.5600 295.9100 0) (fields_autoplaced yes) (effects (font (size 1.27 1.27)) (justify left)) (property "Intersheetrefs" "${INTERSHEET_REFS}" (at 292.1000 295.9100 0) (effects (font (size 1.27 1.27)) (justify left) (hide yes))))
+	(global_label "BOOTSEL_SWITCH" (shape bidirectional) (at 289.5600 300.9900 0) (fields_autoplaced yes) (effects (font (size 1.27 1.27)) (justify left)) (property "Intersheetrefs" "${INTERSHEET_REFS}" (at 292.1000 300.9900 0) (effects (font (size 1.27 1.27)) (justify left) (hide yes))))
 )
