File: hardware/v2/sheets/05_reference_lo.kicad_sch (KiCad schematic)
At the start: 57 parts, among them U40 LMX2592RHAT, U41 ADF4360-1BCPZ, U42 CDCLVC1104PWR, Y40 SiT8209AC-23-33E-100.000000X

Commit message: hardware: checkpoint corrected V2 routing at 108 opens
Parts:
- added R152: 150R_1%, Resistor_SMD:R_0402_1005Metric, symbol Device:R_Small
- C205: value 15nF_C0G -> 470pF_C0G
- C71: value 100nF -> 100nF_C0G; footprint Capacitor_SMD:C_0402_1005Metric -> Capacitor_SMD:C_1206_3216Metric
- C74: value 1nF_C0G -> 470pF_C0G
- C75: value 3.3nF_C0G -> 22nF_C0G; footprint Capacitor_SMD:C_0402_1005Metric -> Capacitor_SMD:C_0805_2012Metric
- R50: value 33R -> 150R_1%
- R56: value 68R_1% -> 220R_1%
- R59: value 620R_1% -> 1k_1%
- R93: value 51R -> 220R_1%
- U42: footprint Package_SO:TSSOP-8_3x3mm_P0.65mm -> Package_SO:TSSOP-8_4.4x3mm_P0.65mm
Connections:
- net LMX_CPOUT is gone; now on net LMX_VTUNE: C70.1, R56.1, U40.12 (CPout)
- net ADF_CPOUT: now also R93.1
- net ADF_LF1: no longer R93.1
- net GND: now also R152.2
- net LMX_REF_PRE: now also R152.1
- net LMX_VTUNE: no longer C71.1, R56.2
- new net LMX_LF_DAMP: C71.1, R56.2
Other:
- note added: "100 MHz reference, LMX2592 and fixed 2.400 GHz LO See HARDWARE_VALIDATION.md and hardware/v2/README.md for design limits."
- note removed: "100 MHz reference, LMX2592 and fixed 2.410 GHz LO See HARDWARE_VALIDATION.md and hardware/v2/README.md for design limits."
- title: 05 - 100 MHz reference, LMX2592 and fixed 2.410 GHz LO -> 05 - 100 MHz reference, LMX2592 and fixed 2.400 GHz LO
Changed lines of the file:
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@@
 	(paper "A1")
 	(title_block
-		(title "05 - 100 MHz reference, LMX2592 and fixed 2.410 GHz LO")
+		(title "05 - 100 MHz reference, LMX2592 and fixed 2.400 GHz LO")
 		(rev "2.0")
 		(company "Code-SDR")
@@
 			)
 		)
-		(property "Footprint" "Package_SO:TSSOP-8_3x3mm_P0.65mm"
+		(property "Footprint" "Package_SO:TSSOP-8_4.4x3mm_P0.65mm"
 			(at 180.34 90.17 0.0000)
 			(effects
@@
 			)
 		)
-		(property "Value" "33R"
+		(property "Value" "150R_1%"
 			(at 291.338 90.17 90)
 			(effects
@@
 			)
 		)
-		(property "Description" "LMX_CPOUT local bypass"
+		(property "Description" "LMX_VTUNE local bypass"
 			(at 400.05 350.52 0)
 			(effects
@@
 			)
 		)
-		(property "Value" "68R_1%"
+		(property "Value" "220R_1%"
 			(at 512.318 350.52 90)
 			(effects
@@
 			)
 		)
-		(property "Value" "100nF"
+		(property "Value" "100nF_C0G"
 			(at 620.014 348.488 0.0000)
 			(effects
@@
 			)
 		)
-		(property "Footprint" "Capacitor_SMD:C_0402_1005Metric"
+		(property "Footprint" "Capacitor_SMD:C_1206_3216Metric"
 			(at 619.76 350.52 0.0000)
 			(effects
@@
 			)
 		)
-		(property "Description" "LMX_VTUNE local bypass"
+		(property "Description" "LMX_LF_DAMP local bypass"
 			(at 619.76 350.52 0)
 			(effects
@@
 			)
 		)
-		(property "Description" "Fixed 2.410 GHz integer-N second LO: 100 MHz/R20, P16, B30, A2"
+		(property "Description" "Fixed 2.400 GHz integer-N second LO: 100 MHz/R20, P16, B30, A0"
 			(at 730.25 350.52 0)
 			(effects
@@
 			)
 		)
-		(property "Value" "1nF_C0G"
+		(property "Value" "470pF_C0G"
 			(at 400.304 400.558 0.0000)
 			(effects
@@
 			)
 		)
-		(property "Value" "620R_1%"
+		(property "Value" "1k_1%"
 			(at 512.318 402.59 90)
 			(effects
@@
 			)
 		)
-		(property "Value" "3.3nF_C0G"
+		(property "Value" "22nF_C0G"
 			(at 620.014 400.558 0.0000)
 			(effects
@@
 			)
 		)
-		(property "Footprint" "Capacitor_SMD:C_0402_1005Metric"
+		(property "Footprint" "Capacitor_SMD:C_0805_2012Metric"
 			(at 619.76 402.59 0.0000)
 			(effects
@@
 			)
 		)
-		(property "Value" "51R"
+		(property "Value" "220R_1%"
 			(at 732.028 402.59 90)
 			(effects
@@
 			)
 		)
-		(property "Value" "15nF_C0G"
+		(property "Value" "470pF_C0G"
 			(at 70.104 451.358 0.0000)
 			(effects
@@
 		(at 422.91 140.97)
 	)
-	(text "100 MHz reference, LMX2592 and fixed 2.410 GHz LO\nSee HARDWARE_VALIDATION.md and hardware/v2/README.md for design limits."
+	(text "100 MHz reference, LMX2592 and fixed 2.400 GHz LO\nSee HARDWARE_VALIDATION.md and hardware/v2/README.md for design limits."
 		(exclude_from_sim no)
 		(at 150 25 0.0000)
@@
 		)
 	)
-	(global_label "LMX_CPOUT"
+	(global_label "LMX_VTUNE"
 		(shape bidirectional)
 		(at 377.1900 143.5100 0)
@@
 		)
 	)
-	(global_label "LMX_CPOUT"
+	(global_label "LMX_VTUNE"
 		(shape bidirectional)
 		(at 400.0500 347.9800 0)
@@
 		)
 	)
-	(global_label "LMX_CPOUT"
+	(global_label "LMX_VTUNE"
 		(shape bidirectional)
 		(at 510.5400 347.9800 0)
@@
 		)
 	)
-	(global_label "LMX_VTUNE"
+	(global_label "LMX_LF_DAMP"
 		(shape bidirectional)
 		(at 510.5400 353.0600 0)
@@
 		)
 	)
-	(global_label "LMX_VTUNE"
+	(global_label "LMX_LF_DAMP"
 		(shape bidirectional)
 		(at 619.7600 347.9800 0)
@@
 		)
 	)
-	(global_label "ADF_LF1"
+	(global_label "ADF_CPOUT"
 		(shape bidirectional)
 		(at 730.2500 400.0500 0)
@@
 		)
 	)
+	(symbol (lib_id "Device:R_Small") (at 180.3400 505.4600 0) (unit 1)
+	(exclude_from_sim no) (in_bom yes) (on_board yes)
+	(dnp no)
+	(fields_autoplaced no)
+	(property "Reference" "R152" (at 185.4200 502.9200 0) (effects (font (size 1.27 1.27)) (justify left)))
+	(property "Value" "150R_1%" (at 185.4200 508.0000 0) (effects (font (size 1.27 1.27)) (justify left)))
+	(property "Footprint" "Resistor_SMD:R_0402_1005Metric" (at 185.4200 508.0000 0) (effects (font (size 1.27 1.27)) (justify left) (hide yes)))
+	(property "Datasheet" "" (at 185.4200 508.0000 0) (effects (font (size 1.27 1.27)) (justify left) (hide yes)))
+	(property "Description" "" (at 185.4200 508.0000 0) (effects (font (size 1.27 1.27)) (justify left) (hide yes)))
+	(pin "1")
+	(pin "2")
+	(instances (project "Code-SDR-V2" (path "/b04744a4-fe39-4740-81de-d5e094f9e157/9a37ff5a-0b61-4e4c-bd9a-14ccc376e131" (reference "R152") (unit 1))))
+)
+	(global_label "LMX_REF_PRE" (shape bidirectional) (at 180.3400 502.9200 0) (fields_autoplaced yes) (effects (font (size 1.27 1.27)) (justify left)) (property "Intersheetrefs" "${INTERSHEET_REFS}" (at 182.8800 502.9200 0) (effects (font (size 1.27 1.27)) (justify left) (hide yes))))
+	(global_label "GND" (shape bidirectional) (at 180.3400 508.0000 0) (fields_autoplaced yes) (effects (font (size 1.27 1.27)) (justify left)) (property "Intersheetrefs" "${INTERSHEET_REFS}" (at 182.8800 508.0000 0) (effects (font (size 1.27 1.27)) (justify left) (hide yes))))
 )
