File: hardware/v2/sheets/07_rf_high.kicad_sch (KiCad schematic)
At the start: 53 parts, among them J60 RF_HIGH_2.3_4.2GHz, J61 RF_HIGH_4.2_6.8GHz, J62 RF_HIGH_6.8_9.2GHz, J63 RF_HIGH_8.0_10GHz, T60 TC1-1-13M+, U60 GRF4001, U61 GRF2101, U62 GRF2101, U63 LTC5548IUDB, U64 QPC6144TR13, U66 GRF2101, U67 GRF2101

Commit message: hardware: checkpoint corrected V2 routing at 108 opens
Parts:
- added R160, R161: 1k_1%, Resistor_SMD:R_0402_1005Metric, symbol Device:R_Small
- R144, R145: value 100k -> 10k_1%
Connections:
- net HSW_V1: now also R160.1; no longer R144.1, U64.17 (V1)
- net HSW_V2: now also R161.1; no longer R145.1, U64.18 (V2)
- new net HSW_V1_CHIP: R144.1, R160.2, U64.17 (V1)
- new net HSW_V2_CHIP: R145.1, R161.2, U64.18 (V2)
Changed lines of the file:
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@@
 			)
 		)
-		(property "Description" "50 MHz to 12 GHz high-isolation SP4T after the branch LNAs; LC0/LC1 low select 1.8 V logic and V3/VSS are grounded"
+		(property "Description" "50 MHz to 10 GHz high-isolation SP4T after the branch LNAs; LC0/LC1 low select 1.8 V logic and V3/VSS are grounded"
 			(at 69.85 402.59 0)
 			(effects
@@
 			)
 		)
-		(property "Value" "100k"
+		(property "Value" "10k_1%"
 			(at 401.828 402.59 90)
 			(effects
@@
 			)
 		)
-		(property "Value" "100k"
+		(property "Value" "10k_1%"
 			(at 512.318 402.59 90)
 			(effects
@@
 		)
 	)
-	(global_label "HSW_V1"
+	(global_label "HSW_V1_CHIP"
 		(shape bidirectional)
 		(at 92.7100 393.7000 0)
@@
 		)
 	)
-	(global_label "HSW_V2"
+	(global_label "HSW_V2_CHIP"
 		(shape bidirectional)
 		(at 92.7100 396.2400 0)
@@
 		)
 	)
-	(global_label "HSW_V1"
+	(global_label "HSW_V1_CHIP"
 		(shape bidirectional)
 		(at 400.0500 400.0500 0)
@@
 		)
 	)
-	(global_label "HSW_V2"
+	(global_label "HSW_V2_CHIP"
 		(shape bidirectional)
 		(at 510.5400 400.0500 0)
@@
 		)
 	)
+	(symbol (lib_id "Device:R_Small") (at 510.5400 453.3900 0) (unit 1)
+	(exclude_from_sim no) (in_bom yes) (on_board yes)
+	(dnp no)
+	(fields_autoplaced no)
+	(property "Reference" "R160" (at 515.6200 450.8500 0) (effects (font (size 1.27 1.27)) (justify left)))
+	(property "Value" "1k_1%" (at 515.6200 455.9300 0) (effects (font (size 1.27 1.27)) (justify left)))
+	(property "Footprint" "Resistor_SMD:R_0402_1005Metric" (at 515.6200 455.9300 0) (effects (font (size 1.27 1.27)) (justify left) (hide yes)))
+	(property "Datasheet" "" (at 515.6200 455.9300 0) (effects (font (size 1.27 1.27)) (justify left) (hide yes)))
+	(property "Description" "" (at 515.6200 455.9300 0) (effects (font (size 1.27 1.27)) (justify left) (hide yes)))
+	(pin "1")
+	(pin "2")
+	(instances (project "Code-SDR-V2" (path "/b04744a4-fe39-4740-81de-d5e094f9e157/04d9fde5-a5d7-4580-9575-937060eadc46" (reference "R160") (unit 1))))
+)
+	(symbol (lib_id "Device:R_Small") (at 619.7600 453.3900 0) (unit 1)
+	(exclude_from_sim no) (in_bom yes) (on_board yes)
+	(dnp no)
+	(fields_autoplaced no)
+	(property "Reference" "R161" (at 624.8400 450.8500 0) (effects (font (size 1.27 1.27)) (justify left)))
+	(property "Value" "1k_1%" (at 624.8400 455.9300 0) (effects (font (size 1.27 1.27)) (justify left)))
+	(property "Footprint" "Resistor_SMD:R_0402_1005Metric" (at 624.8400 455.9300 0) (effects (font (size 1.27 1.27)) (justify left) (hide yes)))
+	(property "Datasheet" "" (at 624.8400 455.9300 0) (effects (font (size 1.27 1.27)) (justify left) (hide yes)))
+	(property "Description" "" (at 624.8400 455.9300 0) (effects (font (size 1.27 1.27)) (justify left) (hide yes)))
+	(pin "1")
+	(pin "2")
+	(instances (project "Code-SDR-V2" (path "/b04744a4-fe39-4740-81de-d5e094f9e157/04d9fde5-a5d7-4580-9575-937060eadc46" (reference "R161") (unit 1))))
+)
+	(global_label "HSW_V1" (shape bidirectional) (at 510.5400 450.8500 0) (fields_autoplaced yes) (effects (font (size 1.27 1.27)) (justify left)) (property "Intersheetrefs" "${INTERSHEET_REFS}" (at 513.0800 450.8500 0) (effects (font (size 1.27 1.27)) (justify left) (hide yes))))
+	(global_label "HSW_V1_CHIP" (shape bidirectional) (at 510.5400 455.9300 0) (fields_autoplaced yes) (effects (font (size 1.27 1.27)) (justify left)) (property "Intersheetrefs" "${INTERSHEET_REFS}" (at 513.0800 455.9300 0) (effects (font (size 1.27 1.27)) (justify left) (hide yes))))
+	(global_label "HSW_V2" (shape bidirectional) (at 619.7600 450.8500 0) (fields_autoplaced yes) (effects (font (size 1.27 1.27)) (justify left)) (property "Intersheetrefs" "${INTERSHEET_REFS}" (at 622.3000 450.8500 0) (effects (font (size 1.27 1.27)) (justify left) (hide yes))))
+	(global_label "HSW_V2_CHIP" (shape bidirectional) (at 619.7600 455.9300 0) (fields_autoplaced yes) (effects (font (size 1.27 1.27)) (justify left)) (property "Intersheetrefs" "${INTERSHEET_REFS}" (at 622.3000 455.9300 0) (effects (font (size 1.27 1.27)) (justify left) (hide yes))))
 )
