File: hardware/v2/sheets/08_if_chain.kicad_sch (KiCad schematic)
At the start: 56 parts, among them T70 2450BL15B0100001E, U70 BGS12WN6E6327, U71 GRF2013, U72 PE4312C-Z, U73 LT5560EDD, U74 AD8351ARMZ, U75 GRF2013

Commit message: hardware: checkpoint corrected V2 routing at 108 opens
Parts:
- C262, C268: value 100pF_C0G -> 51pF_C0G
- C264, C266: value 110pF_C0G -> 56pF_C0G
Connections:
- net +3V3_ANA: now also U73.2 (EN)
- net +3V3_DIG: no longer U73.2 (EN)
Other:
- note added: "2.42625 GHz IF, DSA, second mixer and ADC driver See HARDWARE_VALIDATION.md and hardware/v2/README.md for design limits."
- note removed: "2.43625 GHz IF, DSA, second mixer and ADC driver See HARDWARE_VALIDATION.md and hardware/v2/README.md for design limits."
- title: 08 - 2.43625 GHz IF, DSA, second mixer and ADC driver -> 08 - 2.42625 GHz IF, DSA, second mixer and ADC driver
Changed lines of the file:
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@@
 	(paper "A1")
 	(title_block
-		(title "08 - 2.43625 GHz IF, DSA, second mixer and ADC driver")
+		(title "08 - 2.42625 GHz IF, DSA, second mixer and ADC driver")
 		(rev "2.0")
 		(company "Code-SDR")
@@
 			)
 		)
-		(property "Description" "First-IF low/high path selector at 2.43625 GHz"
+		(property "Description" "First-IF low/high path selector at 2.42625 GHz"
 			(at 180.34 90.17 0)
 			(effects
@@
 			)
 		)
-		(property "Description" "2.410 GHz second mixer producing 26.25 MHz center IF"
+		(property "Description" "2.400 GHz second mixer producing 26.25 MHz center IF"
 			(at 289.56 246.38 0)
 			(effects
@@
 			)
 		)
-		(property "Value" "100pF_C0G"
+		(property "Value" "51pF_C0G"
 			(at 620.014 348.488 0.0000)
 			(effects
@@
 			)
 		)
-		(property "Value" "110pF_C0G"
+		(property "Value" "56pF_C0G"
 			(at 730.504 348.488 0.0000)
 			(effects
@@
 			)
 		)
-		(property "Value" "110pF_C0G"
+		(property "Value" "56pF_C0G"
 			(at 70.104 400.558 0.0000)
 			(effects
@@
 			)
 		)
-		(property "Value" "100pF_C0G"
+		(property "Value" "51pF_C0G"
 			(at 180.594 400.558 0.0000)
 			(effects
@@
 		(at 753.11 189.23)
 	)
-	(text "2.43625 GHz IF, DSA, second mixer and ADC driver\nSee HARDWARE_VALIDATION.md and hardware/v2/README.md for design limits."
+	(text "2.42625 GHz IF, DSA, second mixer and ADC driver\nSee HARDWARE_VALIDATION.md and hardware/v2/README.md for design limits."
 		(exclude_from_sim no)
 		(at 150 25 0.0000)
@@
 		)
 	)
-	(global_label "+3V3_DIG"
+	(global_label "+3V3_ANA"
 		(shape bidirectional)
 		(at 266.7000 238.7600 0)
