File: hardware/v2/Code-SDR-V2.kicad_pcb (KiCad board)
At the start: 4 copper layers, 101.6 x 101.6 mm, 373 parts, among them J1 5V_INPUT_ONLY, J10 USB_B_Micro, J11 Cortex_SWD_10pin, J30 JK0654219NL, J50 RF_LOW_0.01_2.5GHz_OPTION, J60 RF_HIGH_2.3_4.2GHz, J61 RF_HIGH_4.2_6.8GHz, J62 RF_HIGH_6.8_9.2GHz, J63 RF_HIGH_8.0_10GHz, SW1 BOOTSEL, SW2 RESET, T50 2450BL15B0200001E, T60 TC1-1-13M+, T70 2450BL15B0100001E, U1 TLV62569DBVR, U10 RP2040, U11 W25Q16JVSNIQ, U12 USBLC6-2SC6, U2 TLV62569DBVR, U20 LIF-MD6000-6JMG80I, U21 AD9215BCPZ-105, U3 TLV75525PDBVR, U30 KSZ9031RNXCA, U4 TPS7A8300ARGWT, U40 LMX2592RHAT, U41 ADF4360-1BCPZ, U42 CDCLVC1104PWR, U5 TPS389033DSER, U50 GRF4001, U51 ADL5801ACPZ-R7, U6 TPS389033DSER, U60 GRF4001, U61 GRF2101, U62 GRF2101, U63 LTC5548IUDB, U64 QPC6144TR13, U66 GRF2101, U67 GRF2101, U7 TPS389033DSER, U70 BGS12WN6E6327, U71 GRF2013, U72 PE4312C-Z, U73 LT5560EDD, U74 AD8351ARMZ, U75 GRF2013, U8 TPS389012DSER, U9 TPS389012DSER, Y10 ABM8-272-T3_12MHz, Y30 ECS-250-20-33-TR_25MHz, Y40 SiT8209AC-23-33E-100.000000X

Commit message: hardware: connect twelve FPGA IO rail groups
Routing:
- net FPGA_VCCIO0_3V3: track 51.8 -> 62.3 mm, vias 15 -> 16
- net FPGA_VCCIO2_3V3: track 29.3 -> 36.7 mm, vias 6 -> 8
- net FPGA_VCCIO1_3V3: track 43.9 -> 45.1 mm

Commit message: hardware: close ten short Code-SDR gaps
Routing:
- net SW_1V2: track 8.64 -> 15.5 mm
- net PHY_AVDDH_3V3: track 39.2 -> 42.2 mm
- net FPGA_PLL_1V2: track 27.5 -> 30.3 mm
- net FB_ANA: track 1.21 -> 3.59 mm
- net GND: track 245.2 -> 247.0 mm
- net ADC_REFT: track 1.73 -> 2.96 mm
- net ADC_REFB: track 1.40 -> 2.57 mm
- net CORE_EN: track 45.2 -> 46.3 mm
- net PHY_PLL_1V2: track 7.53 -> 8.43 mm
Changed lines of the file:
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@@
 	)
 	(segment
+		(start 75.4018 68.9)
+		(end 75 68.9)
+		(width 0.1)
+		(layer "F.Cu")
+		(net 26)
+	)
+	(segment
+		(start 75.40182 69.67007)
+		(end 75.4018 68.9)
+		(width 0.1)
+		(layer "F.Cu")
+		(net 26)
+	)
+	(segment
 		(start 72.5 69.3261)
 		(end 73.2391 69.32615)
@@
 	(segment
 		(start 74.5982 67)
+		(end 74.0336 67.2455)
+		(width 0.1)
+		(layer "F.Cu")
+		(net 27)
+	)
+	(segment
+		(start 74.5982 67)
 		(end 74.59818 65.82993)
 		(width 0.1)
@@
 		(net 27)
 	)
+	(segment
+		(start 74.0336 67.2455)
+		(end 73.7391 67.78615)
+		(width 0.1)
+		(layer "F.Cu")
+		(net 27)
+	)
 	(via
 		(at 71.2391 67.57615)
@@
 	)
 	(segment
+		(start 50.3425 64.774199)
+		(end 50.502476 64.774203)
+		(width 0.1)
+		(layer "F.Cu")
+		(net 58)
+	)
+	(segment
 		(start 54.742476 60.294203)
 		(end 50.662476 64.374202)
@@
 	)
 	(segment
+		(start 50.342476 65.094201)
+		(end 50.3425 64.774199)
+		(width 0.1)
+		(layer "F.Cu")
+		(net 58)
+	)
+	(segment
 		(start 50.815514 64.552476)
 		(end 50.755514 64.552476)
@@
 	)
 	(segment
+		(start 56.32615 75.2391)
+		(end 57.5323 75.9298)
+		(width 0.1)
+		(layer "F.Cu")
+		(net 60)
+	)
+	(segment
 		(start 55.175169 62.255823)
 		(end 55.115169 62.315823)
@@
 		(net 60)
 	)
+	(segment
+		(start 57.5323 75.9298)
+		(end 58.18 74.7)
+		(width 0.1)
+		(layer "F.Cu")
+		(net 60)
+	)
 	(via
 		(at 55.415169 61.955823)
@@
 	)
 	(segment
+		(start 53.92007 66.40182)
+		(end 52.95 66.401799)
+		(width 0.1)
+		(layer "F.Cu")
+		(net 71)
+	)
+	(segment
 		(start 16.52 37.32)
 		(end 15.52 36.32)
@@
 	)
 	(segment
+		(start 52.95 66.401799)
+		(end 52.95 65.599999)
+		(width 0.1)
+		(layer "F.Cu")
+		(net 71)
+	)
+	(segment
 		(start 33.205 58.981347)
 		(end 33.205 59.221347)
@@
 	)
 	(segment
+		(start 83.9691 77.08)
+		(end 83.9691 74.94385)
+		(width 0.1)
+		(layer "F.Cu")
+		(net 158)
+	)
+	(segment
 		(start 76.225 76.19)
 		(end 76.67 76.19)
@@
 	)
 	(segment
+		(start 83.18 77.08)
+		(end 83.9691 77.08)
+		(width 0.1)
+		(layer "F.Cu")
+		(net 158)
+	)
+	(segment
 		(start 84.823895 58.668885)
 		(end 81.943895 61.548885)
@@
 	)
 	(segment
+		(start 84.38 69.6739)
+		(end 85.0109 69.67385)
+		(width 0.1)
+		(layer "F.Cu")
+		(net 165)
+	)
+	(segment
 		(start 85.88 69.89)
 		(end 85.88 70.88)
@@
 	)
 	(segment
+		(start 84.38 69.4)
+		(end 84.38 69.6739)
+		(width 0.1)
+		(layer "F.Cu")
+		(net 165)
+	)
+	(segment
 		(start 86.55 68.695)
 		(end 86.55 69.22)
@@
 	)
 	(segment
+		(start 7.0925 72.88)
+		(end 5.41 75.88)
+		(width 0.1)
+		(layer "F.Cu")
+		(net 239)
+	)
+	(segment
 		(start 5.41 75.88)
 		(end 4.854 76.436)
@@
 	)
 	(segment
+		(start 8.775 75.88)
+		(end 7.0925 72.88)
+		(width 0.1)
+		(layer "F.Cu")
+		(net 239)
+	)
+	(segment
 		(start 3.565 86.88)
 		(end 3.285 86.6)
@@
 	)
 	(segment
+		(start 7.21 75.8)
+		(end 7.41 76.3)
+		(width 0.1)
+		(layer "F.Cu")
+		(net 253)
+	)
+	(segment
 		(start 25.378765 68.637312)
 		(end 25.458765 68.557312)
@@
 	)
 	(segment
+		(start 7.41 75.3)
+		(end 7.21 75.8)
+		(width 0.1)
+		(layer "F.Cu")
+		(net 253)
+	)
+	(segment
 		(start 24.738765 68.877312)
 		(end 24.818765 68.877312)
@@
 	)
 	(segment
+		(start 20.1618 87.9752)
+		(end 19.22 88.7)
+		(width 0.1)
+		(layer "F.Cu")
+		(net 254)
+	)
+	(segment
 		(start 22.773628 90.065514)
 		(end 22.453628 90.065514)
@@
 		(layer "F.Cu")
 		(net 254)
+	)
+	(segment
+		(start 21.14 88.65)
+		(end 20.1618 87.9752)
+		(width 0.1)
+		(layer "F.Cu")
+		(net 254)
